File: PT2399.sch (KiCad schematic (older format))
At the start: 33 parts, among them J1 Output Jack, J2 Input Jack, J3 Jack-DC, Q101 2N2219, Q102 2N2219, SW101 SW_SPST, U1 L78L05_TO92, U101 4066, U102 4049, U3 TL072

Commit message: Needed an extra coupling cap I guess
Parts:
- added C?: 1u, symbol Device:C
Connections:
- net delay_out: now also C?.1; no longer RV102.2
- new net: C?.2, RV102.2
Other:
- moved on the sheet: Q101, Q102, RV103
Changed lines of the file:
@@
 F4 "time" O R 3800 4650 50
 $EndSheet
-Text GLabel 6500 5000 2    50   Output ~ 0
+Text GLabel 6900 5000 2    50   Output ~ 0
 delay_out
 $Comp
@@
 Wire Wire Line
 	6200 5250 6200 5150
-Wire Wire Line
-	6500 5000 6350 5000
 $Comp
 L Device:CP C102
@@
 L Transistor_BJT:2N2219 Q101
 U 1 1 5F998DE9
-P 7600 5450
-F 0 "Q101" H 7791 5496 50  0000 L CNN
-F 1 "2N2219" H 7791 5405 50  0000 L CNN
-F 2 "Package_TO_SOT_THT:TO-39-3" H 7800 5375 50  0001 L CIN
-F 3 "http://www.onsemi.com/pub_link/Collateral/2N2219-D.PDF" H 7600 5450 50  0001 L CNN
-	1    7600 5450
+P 9450 5050
+F 0 "Q101" H 9641 5096 50  0000 L CNN
+F 1 "2N2219" H 9641 5005 50  0000 L CNN
+F 2 "Package_TO_SOT_THT:TO-39-3" H 9650 4975 50  0001 L CIN
+F 3 "http://www.onsemi.com/pub_link/Collateral/2N2219-D.PDF" H 9450 5050 50  0001 L CNN
+	1    9450 5050
 	-1   0    0    -1
 $EndComp
@@
 L Device:R_POT RV103
 U 1 1 5F99A658
-P 7500 4900
+P 9350 4500
 AR Path="/5F99A658" Ref="RV103"  Part="1"
 AR Path="/5F90D1E6/5F99A658" Ref="RV?"  Part="1"
 AR Path="/5F9672E5/5F99A658" Ref="RV?"  Part="1"
-F 0 "RV103" V 7293 4900 50  0000 C CNN
-F 1 "b50k" V 7384 4900 50  0000 C CNN
-F 2 "" H 7500 4900 50  0001 C CNN
-F 3 "~" H 7500 4900 50  0001 C CNN
-	1    7500 4900
-	1    0    0    -1
-$EndComp
-Wire Wire Line
-	7650 4900 7650 4750
-Wire Wire Line
-	7650 4750 7500 4750
+F 0 "RV103" V 9143 4500 50  0000 C CNN
+F 1 "b50k" V 9234 4500 50  0000 C CNN
+F 2 "" H 9350 4500 50  0001 C CNN
+F 3 "~" H 9350 4500 50  0001 C CNN
+	1    9350 4500
+	1    0    0    -1
+$EndComp
+Wire Wire Line
+	9500 4500 9500 4350
+Wire Wire Line
+	9500 4350 9350 4350
 Text Label 3900 4650 0    50   ~ 0
 time1
@@
 	4800 4650 4700 4650
 Wire Wire Line
-	7500 5050 7500 5150
-Text Label 7500 4600 1    50   ~ 0
+	9350 4650 9350 4750
+Text Label 9350 4200 1    50   ~ 0
 time1
 Wire Wire Line
-	7500 4600 7500 4750
-Connection ~ 7500 4750
+	9350 4200 9350 4350
+Connection ~ 9350 4350
 $Comp
 L power:GND #PWR0104
 U 1 1 5F9B9107
-P 7500 5800
-F 0 "#PWR0104" H 7500 5550 50  0001 C CNN
-F 1 "GND" H 7505 5627 50  0000 C CNN
-F 2 "" H 7500 5800 50  0001 C CNN
-F 3 "" H 7500 5800 50  0001 C CNN
-	1    7500 5800
-	1    0    0    -1
-$EndComp
-Wire Wire Line
-	7500 5800 7500 5650
-Connection ~ 7500 5150
-Wire Wire Line
-	7500 5150 7500 5250
+P 9350 5400
+F 0 "#PWR0104" H 9350 5150 50  0001 C CNN
+F 1 "GND" H 9355 5227 50  0000 C CNN
+F 2 "" H 9350 5400 50  0001 C CNN
+F 3 "" H 9350 5400 50  0001 C CNN
+	1    9350 5400
+	1    0    0    -1
+$EndComp
+Wire Wire Line
+	9350 5400 9350 5250
+Connection ~ 9350 4750
+Wire Wire Line
+	9350 4750 9350 4850
 $Comp
 L Transistor_BJT:2N2219 Q102
 U 1 1 5F9BD375
-P 8100 5450
-F 0 "Q102" H 8290 5496 50  0000 L CNN
-F 1 "2N2219" H 8290 5405 50  0000 L CNN
-F 2 "Package_TO_SOT_THT:TO-39-3" H 8300 5375 50  0001 L CIN
-F 3 "http://www.onsemi.com/pub_link/Collateral/2N2219-D.PDF" H 8100 5450 50  0001 L CNN
-	1    8100 5450
-	1    0    0    -1
-$EndComp
-Wire Wire Line
-	7900 5450 7850 5450
-Wire Wire Line
-	7850 5450 7850 5150
-Wire Wire Line
-	7500 5150 7850 5150
-Connection ~ 7850 5450
-Wire Wire Line
-	7850 5450 7800 5450
+P 9950 5050
+F 0 "Q102" H 10140 5096 50  0000 L CNN
+F 1 "2N2219" H 10140 5005 50  0000 L CNN
+F 2 "Package_TO_SOT_THT:TO-39-3" H 10150 4975 50  0001 L CIN
+F 3 "http://www.onsemi.com/pub_link/Collateral/2N2219-D.PDF" H 9950 5050 50  0001 L CNN
+	1    9950 5050
+	1    0    0    -1
+$EndComp
+Wire Wire Line
+	9750 5050 9700 5050
+Wire Wire Line
+	9700 5050 9700 4750
+Wire Wire Line
+	9350 4750 9700 4750
+Connection ~ 9700 5050
+Wire Wire Line
+	9700 5050 9650 5050
 $Comp
 L power:GND #PWR0105
 U 1 1 5F9C2DE0
-P 8200 5800
-F 0 "#PWR0105" H 8200 5550 50  0001 C CNN
-F 1 "GND" H 8205 5627 50  0000 C CNN
-F 2 "" H 8200 5800 50  0001 C CNN
-F 3 "" H 8200 5800 50  0001 C CNN
-	1    8200 5800
-	1    0    0    -1
-$EndComp
-Wire Wire Line
-	8200 5800 8200 5650
-Text Label 8200 5000 1    50   ~ 0
+P 10050 5400
+F 0 "#PWR0105" H 10050 5150 50  0001 C CNN
+F 1 "GND" H 10055 5227 50  0000 C CNN
+F 2 "" H 10050 5400 50  0001 C CNN
+F 3 "" H 10050 5400 50  0001 C CNN
+	1    10050 5400
+	1    0    0    -1
+$EndComp
+Wire Wire Line
+	10050 5400 10050 5250
+Text Label 10050 4600 1    50   ~ 0
 time2
 Wire Wire Line
-	8200 5000 8200 5250
+	10050 4600 10050 4850
 Text GLabel 3400 5750 2    50   Input ~ 0
 !freeze
@@
 Wire Wire Line
 	4500 5250 5250 5250
+$Comp
+L Device:C C?
+U 1 1 5FB6414D
+P 6600 5000
+F 0 "C?" V 6348 5000 50  0000 C CNN
+F 1 "1u" V 6439 5000 50  0000 C CNN
+F 2 "" H 6638 4850 50  0001 C CNN
+F 3 "~" H 6600 5000 50  0001 C CNN
+	1    6600 5000
+	0    1    1    0
+$EndComp
+Wire Wire Line
+	6900 5000 6750 5000
+Wire Wire Line
+	6450 5000 6350 5000
 $EndSCHEMATC
